Commit message: feat: TCP 를 손가락 가운데로 — GripperDA_v2 [0, 2.7, 228] · rg2_tcp x −2.7 mm · 공급 칸 y +2.7 mm (10/8 PL A안)
손가락 가운데가 GripperDA_v1(J6 축 위)에서 rg2_tcp −x(플랜지 +y) 2.7 mm 비켜 있어, 손목을 돌려 놓는 블록이 3~6 mm 어긋났다(004 시험으로 확인).
TCP 정의 자체를 손가락 가운데로 옮겨 집기 · 놓기 · 카메라 집기에 한 곳에서 들어가게 한다. 공급 칸은 옛 TCP 로 맞춘 좌표라 같은 손가락 위치로 집게 옮김.

변경 파일: src/d2_robot/d2_bringup/config/tcp.json, src/d2_robot/d2_bringup/config/robot.yaml, src/d2_robot/d2_bringup/description/m0609_rg2_tcp.urdf.xacro, src/d2_robot/d2_bringup/launch/real_moveit.launch.py, src/d2_robot/d2_motion/d2_motion/motion_math.py
영향: 로봇 동작(브링업 TCP · 공급 칸), 비전(손목 보정은 이 PR merge 뒤 민범진 — tcp.json 이름 비교). 제어기에 GripperDA_v2 등록 · 활성화 전에는 pick_place 가 목표를 거절함

File: src/d2_robot/d2_bringup/description/m0609_rg2_tcp.urdf.xacro (robot description, xacro)
@@ -6,7 +6,12 @@
          rg2_base_link 원점은 플랜지에서 공구 축으로 4 mm 이므로, 플랜지 -> 손가락 끝 = tcp_z + 0.004.
          기본 0.224 = 플랜지 -> 손가락 끝 228 mm (작업 2 TCP 값). 실측값이 다르면 바꾼다.
+  tcp_x · tcp_y: 손가락 가운데가 공구 축에서 옆으로 비켜난 양 (m, rg2_tcp 틀 — y = 닫힘 방향). 기본 0.
+         브링업(real_moveit.launch.py)이 config/tcp.json 에서 tcp_z 와 함께 넘긴다 — 10/8: 손목을 돌리면 손가락 가운데가
+         회전축에서 비켜 있어 놓는 블록이 어긋남(004 실기), x -2.7 mm (PL A안).
 -->
 <robot xmlns:xacro="http://ros.org/wiki/xacro" name="m0609_rg2_camera">
   <xacro:arg name="tcp_z" default="0.224"/>
+  <xacro:arg name="tcp_x" default="0.0"/>
+  <xacro:arg name="tcp_y" default="0.0"/>
   <xacro:include filename="$(find m0609_rg2_bringup)/urdf/m0609_with_rg2_camera.urdf.xacro"/>
   <link name="rg2_tcp"/>
@@ -14,5 +19,5 @@
     <parent link="rg2_base_link"/>
     <child link="rg2_tcp"/>
-    <origin xyz="0 0 $(arg tcp_z)" rpy="0 0 0"/>
+    <origin xyz="$(arg tcp_x) $(arg tcp_y) $(arg tcp_z)" rpy="0 0 0"/>
   </joint>
 </robot>
