Commit message: feat: E-81 손끝 = 손가락 가운데 — 펜던트 GripperDA_v1 값 [0, 2.7, 228] 편집 · 브링업 rg2_tcp x −2.7 · 공급 칸 y +2.7 (진행: W149, 10/10 PL)
E-70 방법을 PL이 10/10 정함(결정 1): 새 이름 등록 대신 펜던트의 기존 GripperDA_v1 값을 손가락 가운데로 편집,
tcp.json 한 곳이 정본 — 브링업이 MoveIt rg2_tcp를 여기서 만든다(박진용 94f8c09 코드 + 이름 v1, finger.center_offset_m 없음).
10/9까지의 posx 기록 · 손목 보정값은 옛 v1 [0, 0, 228] 기준(tcp.json source에 기록). 복구 절차 4절에 그리퍼 응답 없음 때 순서(결정 4).

변경 파일: src/d2_robot/d2_bringup/config/tcp.json, src/d2_robot/d2_bringup/config/robot.yaml, src/d2_robot/d2_bringup/description/m0609_rg2_tcp.urdf.xacro, src/d2_robot/d2_bringup/launch/real_moveit.launch.py, src/d2_robot/d2_motion/d2_motion/motion_math.py, docs/02_인터페이스_IRD_v3_101008.md, docs/01_요구사항_BR-SR_v3_101008.md, docs/복구절차_정지뒤다시시작_v1_101008.md, docs/decisions/결정기록_PC배치_MQTT_CI_1006_v1_101008.md, docs/decisions/README.md, CHANGES.md, web/README.md · web/backend/README.md(링크만)
영향: 로봇 동작(브링업 TCP · 공급 칸 6곳) · 비전(손목 보정은 W156에서 새 기준으로) — 펜던트 편집 뒤 브링업, 3동작 확인 뒤 merge

Co-Authored-By: Claude Opus 5.5 <noreply@anthropic.com>

File: src/d2_robot/d2_bringup/description/m0609_rg2_tcp.urdf.xacro (robot description, xacro)
@@ -6,7 +6,12 @@
          rg2_base_link 원점은 플랜지에서 공구 축으로 4 mm 이므로, 플랜지 -> 손가락 끝 = tcp_z + 0.004.
          기본 0.224 = 플랜지 -> 손가락 끝 228 mm (작업 2 TCP 값). 실측값이 다르면 바꾼다.
+  tcp_x · tcp_y: 손가락 가운데가 공구 축에서 옆으로 비켜난 양 (m, rg2_tcp 틀 — y = 닫힘 방향). 기본 0.
+         브링업(real_moveit.launch.py)이 config/tcp.json 에서 tcp_z 와 함께 넘긴다 — 10/8: 손목을 돌리면 손가락 가운데가
+         회전축에서 비켜 있어 놓는 블록이 어긋남(004 실기), x -2.7 mm (10/10 E-81 — 펜던트 GripperDA_v1 값 편집).
 -->
 <robot xmlns:xacro="http://ros.org/wiki/xacro" name="m0609_rg2_camera">
   <xacro:arg name="tcp_z" default="0.224"/>
+  <xacro:arg name="tcp_x" default="0.0"/>
+  <xacro:arg name="tcp_y" default="0.0"/>
   <xacro:include filename="$(find m0609_rg2_bringup)/urdf/m0609_with_rg2_camera.urdf.xacro"/>
   <link name="rg2_tcp"/>
@@ -14,5 +19,5 @@
     <parent link="rg2_base_link"/>
     <child link="rg2_tcp"/>
-    <origin xyz="0 0 $(arg tcp_z)" rpy="0 0 0"/>
+    <origin xyz="$(arg tcp_x) $(arg tcp_y) $(arg tcp_z)" rpy="0 0 0"/>
   </joint>
 </robot>
